Commit message: finished pa2 1, 2a, and 2b (pid controller with joint 3 and reading joihnt states)

File: ros2_ws/src/scara_description/urdf/scara.urdf (robot description, URDF)
Before this commit: robot scara, 7 links, 6 joints
Joints:
- joint arm_1_attach: origin xyz=0 0 0.45 -> xyz=0 0 0
- joint joint_1: origin xyz=0 0 0.05 -> xyz=0 0 0.5; type revolute -> fixed
- joint joint_2: type revolute -> fixed

Commit message: Update scara.urdf

File: ros2_ws/src/scara_description/urdf/scara.urdf (robot description, URDF)
Before this commit: robot scara, 7 links, 6 joints
Joints:
- joint joint_1: type fixed -> revolute
- joint joint_2: type fixed -> revolute
